File: hardware/load-cell.kicad_pcb (KiCad board)
At the start: 2 copper layers, 30 x 30 mm, 27 parts, among them P1 CON-SENSOR, P2 AKL_5_2, P3 AKL_5_2, U1 M24C64, U2 FAN4860, U3 HX711, U4 DRILL, U5 DRILL, U6 DRILL, U7 DRILL

Commit message: fix weee footprint
Parts:
- removed the VAL at (157.3, 100.1)
- added G***: LOGO, kicad-libraries:WEEE_7mm, B.Cu at (157.3, 100.1)

Commit message: Add 3d information (final); fix orientation of symbols
Parts:
- C1, C2, C3, C4, C5, C6, C7, C8, L2: footprint kicad-libraries:0603 -> kicad-libraries:C0603
- L1: footprint kicad-libraries:0805 -> kicad-libraries:C0805
- R1: footprint kicad-libraries:0603 -> kicad-libraries:R0603
- moved VAL 0.10 mm to (150.8, 100.1)
Connections:
- P1 pad 1: (no net) -> Net-(P1-Pad1)
- U1 pad 7: (no net) -> Net-(U1-Pad7)
- U3 pad 13: (no net) -> Net-(U3-Pad13)
- U3 pad 2: (no net) -> Net-(U3-Pad2)
- U3 pad 6: (no net) -> Net-(U3-Pad6)
Other:
- outline, holes or cut-outs redrawn
